File: pellet_dispenser_controller.kicad_pcb (KiCad board)
At the start: 2 copper layers, 74.9 x 80.6 mm, 105 parts, among them P1 PWR_JACK_2.1x5.5_SMD_RA, SW1 SPDT_SLIDE_500A_SM, U1 DRV103, U2 DRV103, U3 DRV103, U4 DRV103, U5 DRV103, U6 DRV103, U7 DRV103, U8 DRV103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

Commit message: Update names
Parts:
- removed C1: 10uF, pellet_dispenser_controller:SM0805
- removed C10, C12, C14, C16, C18, C2, C4, C6, C8: 1uF, odor_spike_hold:SM0402_POL
- removed C11, C13, C15, C17, C19, C3, C5, C7, C9: 15nF, odor_spike_hold:SM0402
- removed D1: DIODE_SCHOTTKY_45V_10A, pellet_dispenser_controller:CFP15
- removed D10, D12, D14, D16, D18, D20, D4, D6, D8: DIODE_SCHOTTKY_0402, odor_spike_hold:SM0402_POL
- removed D11, D13, D15, D17, D19, D3, D5, D7, D9: DIODE_LOW_REV_CURRENT_0402, odor_spike_hold:SM0402_POL
- removed D2: DIODE_LOW_REV_CURRENT_0402, pellet_dispenser_controller:SM0402_POL
- removed FID1, FID2, FID3, FID4: FIDUCIAL, pellet_dispenser_controller:FIDUCIAL
- removed L1: LED_GRN, pellet_dispenser_controller:LED0805
- removed L10, L2, L3, L4, L5, L6, L7, L8, L9: LED_GRN, odor_spike_hold:LED0805
- removed MH1, MH2, MH3: VAL**, pellet_dispenser_controller:MOUNTING_HOLE_4-40
- removed P1: PWR_JACK_2.1x5.5_SMD_RA, pellet_dispenser_controller:DCJACK_3PAD_SMD_RA
- removed R1: 390, pellet_dispenser_controller:SM0402
- removed R10, R13, R16, R19, R22, R25, R28, R4, R7: 205k, odor_spike_hold:SM0402
- removed R11, R14, R17, R2, R20, R23, R26, R5, R8: 390, odor_spike_hold:SM0402
- removed R12, R15, R18, R21, R24, R27, R3, R6, R9: 150k, odor_spike_hold:SM0402
- removed S1, S2, S3, S4, S5, S6, S7, S8, S9: VAL**, odor_spike_hold:LEECO_LHDB
- removed SW1: SPDT_SLIDE_500A_SM, pellet_dispenser_controller:SPDT_SLIDE_500A_SM
- removed TEENSY1: TEENSY_4.0, pellet_dispenser_controller:TEENSY_4.0
- removed U1, U2, U3, U4, U5, U6, U7, U8, U9: DRV103, odor_spike_hold:SOIC_8
Routing:
- net GND: track 300.6 -> 0.00 mm, vias 1 -> 0
- net VCC: track 286.7 -> 0.00 mm
- net /ARM_0_ODOR_2: track 94.7 -> 0.00 mm
- net /ARM_0_ODOR_1: track 73.0 -> 0.00 mm, vias 1 -> 0
- net /ARM_0_ODOR_0: track 68.3 -> 0.00 mm, vias 1 -> 0
- net /odor_0/SH: track 66.2 -> 0.00 mm
- net /ARM_1_ODOR_2: track 64.0 -> 0.00 mm
- net /Vled: track 63.4 -> 0.00 mm, vias 1 -> 0
- net /odor_2/SH: track 61.2 -> 0.00 mm
- net /ARM_1_ODOR_1: track 59.6 -> 0.00 mm, vias 1 -> 0
- net /odor_1/SH: track 58.7 -> 0.00 mm
- net /odor_8/SH: track 55.0 -> 0.00 mm
- net /ARM_1_ODOR_0: track 53.1 -> 0.00 mm, vias 1 -> 0
- net /odor_7/SH: track 52.7 -> 0.00 mm
- net /odor_5/SH: track 51.8 -> 0.00 mm
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- removed copper zone on B.Cu, net GND
- removed copper zone on F.Cu, net VCC
Other:
- board outline removed
- board text removed: "0"
- board text removed: "1"
- board text removed: "2"
- board text removed: "2.1x5.5 Center + +12VDC"
- board text removed: "ARM"
- board text removed: "ARM 0"
- board text removed: "ARM 1"
- board text removed: "ARM 2"
- board text removed: "ODOR"
- board text removed: "ODOR 0"
- board text removed: "ODOR 1"
- board text removed: "ODOR 2"
- board text removed: "pellet_dispenser_controller Janelia Research Campus 10/2020 ver 1.3"
