File: mouse_reach_controller.kicad_pcb (KiCad board)
At the start: 2 copper layers, 158.8 x 57.2 mm, 51 parts, among them J1 AUDIO_JACK_3.5MM, P1 HEADER_02X05_LATCH, P2 HEADER_02X05_LATCH, P3 HEADER_02X05_LATCH, T1 TERM_BLK_HDR_2POS_90DEG_0.2IN, U1 TMC429, U10 SGTL5000, U2 SN65LVDM050QDRQ1, U3 BUFFER_TRI_STATE_SMALL, U4 SN65LVDM050QDRQ1, U5 BUFFER_TRI_STATE_SMALL, U6 SN65LVDM050QDRQ1, U7 BUFFER_TRI_STATE_SMALL, U8 MIC94091YC6-TR, U9 RT9076-15GV

Commit message: Progress towards v1.1
Connections:
- net /BUZZER_ENABLE renamed /POWER_SWITCH_ENABLE
- net /buzzer_driver/VM renamed /power_switch_driver/VM
Routing:
- net /GND: track 421.3 -> 0.00 mm, vias 4 -> 0
- net /VDD: track 318.1 -> 0.00 mm, vias 4 -> 0
- net /stepper_controller/stepper_driver_interface_2/UART_BUFFERED: track 120.9 -> 0.00 mm, vias 1 -> 0
- net /stepper_controller/stepper_driver_interface_1/UART_BUFFERED: track 85.3 -> 0.00 mm, vias 1 -> 0
- net /~CS: track 79.9 -> 0.00 mm
- net /MISO: track 77.4 -> 0.00 mm
- net /MOSI: track 77.1 -> 0.00 mm
- net /stepper_controller/stepper_driver_interface_0/UART_BUFFERED: track 75.6 -> 0.00 mm
- net /stepper_controller/STEP_2: track 66.7 -> 0.00 mm, vias 2 -> 0
- net /SCK: track 61.3 -> 0.00 mm, vias 1 -> 0
- net /stepper_controller/DIR_2: track 59.9 -> 0.00 mm, vias 2 -> 0
- net /stepper_controller/REF_2: track 52.9 -> 0.00 mm
- net /stepper_controller/REFR_2: track 51.4 -> 0.00 mm
- net /BCLK: track 46.0 -> 0.00 mm
- net /I2S_DIN: track 44.7 -> 0.00 mm, vias 1 -> 0
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- removed copper zone on B.Cu, net /GND
- removed copper zone on F.Cu, net /GND
Other:
- board text added: "Power_Switch"
- board text added: "mouse_reach_controller Janelia Research Campus 11/2021 ver 1.1"
- board text removed: "Buzzer"
- board text removed: "mouse_reach_controller Janelia Research Campus 11/2021 ver 1.0"

Commit message: Add encoder interface
Parts:
- added C17: 0.1uF, mouse_reach_controller:SM0402, F.Cu at (93.8, -9.94)
- added C18: 0.1uF, mouse_reach_controller:SM0402, F.Cu at (93.8, -5.30)
- added D2: DIODE_SCHOTTKY_45V_10A, mouse_reach_controller:CFP15, F.Cu at (227.3, -40.6)
- added P4: HEADER_02X05_LATCH, mouse_reach_controller:HEADER_02x05_LATCH, F.Cu at (389.9, 69.8)
- added P5: HEADER_02X05_LATCH, mouse_reach_controller:HEADER_02x05_LATCH, F.Cu at (384.8, 44.5)
- added P6: PWR_JACK_2.1x5.5_SMD_RA, mouse_reach_controller:DCJACK_3PAD_SMD_RA, F.Cu at (221.0, -58.4)
- added P7: BNC_DOUBLE_RA, mouse_reach_controller:BNC_DOUBLE, F.Cu at (361.9, -83.8)
- added R10: 2.21k, mouse_reach_controller:SM0402, F.Cu at (97.8, -9.94)
- added R9: 2.21k, mouse_reach_controller:SM0402, F.Cu at (95.8, -9.94)
- added T2: TERM_BLK_HDR_4POS_90DEG_0.2IN, mouse_reach_controller:TERM_BLK_HDR_4POS_90DEG_0.2IN, F.Cu at (104.6, -22.0)
- added U11: 74LVC1G125GS, mouse_reach_controller:SOT1202, F.Cu at (99.8, -10.3)
- added U12: 74LVC1G125GS, mouse_reach_controller:SOT1202, F.Cu at (212.1, -94.0)
- C9: value 2.2uF -> 100uF_POL; footprint mouse_reach_controller:SM0402 -> mouse_reach_controller:CP_Elec_6.3x7.7_WURTH
- D1: value DIODE_SCHOTTKY_30V_200mA_0402 -> DIODE_SCHOTTKY_45V_10A; footprint mouse_reach_controller:SM0402_POL -> mouse_reach_controller:CFP15
- FID1, FID2, FID3, FID4: value FIDUCIAL -> FIDUCIAL_1.0mm_MASK2mm; footprint mouse_reach_controller:FIDUCIAL -> mouse_reach_controller:Fiducial_1mm_Mask2mm
- P1, P2: value HEADER_02X05_LATCH -> BNC_DOUBLE_RA; footprint mouse_reach_controller:HEADER_02x05_LATCH -> mouse_reach_controller:BNC_DOUBLE
- U3, U5, U7: value BUFFER_TRI_STATE_SMALL -> 74LVC1G125GS; footprint mouse_reach_controller:MICROPAK2_6LEAD -> mouse_reach_controller:SOT1202
- U8: value MIC94091YC6-TR -> BSP762TXUMA1; footprint mouse_reach_controller:SC70-6 -> mouse_reach_controller:SOIC-8_3.9x4.9mm_P1.27mm
- moved C10 243.1 mm to (340.4, -25.4)
- moved C11 243.1 mm to (340.4, -34.3)
- moved C12 243.1 mm to (340.4, -36.8)
- moved C16 243.1 mm to (331.5, -36.8)
- moved L1 243.1 mm to (340.4, -30.5)
- moved C13 243.1 mm to (330.2, -14.6)
- moved C14 243.1 mm to (330.2, -17.1)
- moved C15 243.1 mm to (330.2, -23.5)
- moved J1 243.1 mm to (330.2, -58.4)
- moved U10 243.1 mm to (330.2, -30.5)
- moved U9 243.1 mm to (330.2, -20.3)
- moved C3 201.1 mm to (337.8, 81.9)
- moved R1 201.1 mm to (332.7, 84.5)
- moved R2 201.1 mm to (332.7, 90.8)
- moved U2 201.1 mm to (337.8, 88.3)
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Connections:
- C9 pad 1: /VCC -> /power_switch_driver/VBB
- P1 pad 1: /stepper_controller/stepper_driver_interface_0/STEP_A -> /BNC_A
- P1 pad 2: /stepper_controller/stepper_driver_interface_0/STEP_B -> /GND
- P1 pad 3: /stepper_controller/stepper_driver_interface_0/DIR_A -> /BNC_B
- P1 pad 4: /stepper_controller/stepper_driver_interface_0/DIR_B -> /GND
- P2 pad 1: /stepper_controller/stepper_driver_interface_1/STEP_A -> /BNC_C
- P2 pad 2: /stepper_controller/stepper_driver_interface_1/STEP_B -> /GND
- P2 pad 3: /stepper_controller/stepper_driver_interface_1/DIR_A -> /BNC_D
- P2 pad 4: /stepper_controller/stepper_driver_interface_1/DIR_B -> /GND
- P3 pad 1: /stepper_controller/stepper_driver_interface_2/STEP_A -> /stepper_controller/stepper_driver_interface_0/STEP_A
- P3 pad 10: /stepper_controller/stepper_driver_interface_2/REFR_B -> /stepper_controller/stepper_driver_interface_0/REFR_B
- P3 pad 2: /stepper_controller/stepper_driver_interface_2/STEP_B -> /stepper_controller/stepper_driver_interface_0/STEP_B
- P3 pad 3: /stepper_controller/stepper_driver_interface_2/DIR_A -> /stepper_controller/stepper_driver_interface_0/DIR_A
- P3 pad 4: /stepper_controller/stepper_driver_interface_2/DIR_B -> /stepper_controller/stepper_driver_interface_0/DIR_B
- P3 pad 5: /stepper_controller/stepper_driver_interface_2/UART_BUFFERED -> /stepper_controller/stepper_driver_interface_0/UART_BUFFERED
- P3 pad 7: /stepper_controller/stepper_driver_interface_2/REF_A -> /stepper_controller/stepper_driver_interface_0/REF_A
- P3 pad 8: /stepper_controller/stepper_driver_interface_2/REF_B -> /stepper_controller/stepper_driver_interface_0/REF_B
- P3 pad 9: /stepper_controller/stepper_driver_interface_2/REFR_A -> /stepper_controller/stepper_driver_interface_0/REFR_A
- TEENSY1 pad 2: (no net) -> /BNC_A
- TEENSY1 pad 3: (no net) -> /BNC_B
- TEENSY1 pad 4: (no net) -> /BNC_C
- TEENSY1 pad 5: (no net) -> /BNC_D
- TEENSY1 pad 6: (no net) -> /ENCODER_A
- TEENSY1 pad 9: (no net) -> /ENCODER_B
- U8 pad 1: /power_switch_driver/VM -> /GND
- U8 pad 2: /GND -> /POWER_SWITCH_ENABLE
- U8 pad 3: (no net) -> /power_switch_driver/VM
- U8 pad 4: /VCC -> (no net)
- U8 pad 5: /GND -> /power_switch_driver/VBB
- U8 pad 6: /POWER_SWITCH_ENABLE -> /power_switch_driver/VBB

Commit message: Progress towards v1.1 layout
Parts:
- added C19: 0.1uF, mouse_reach_controller:SM0402, F.Cu at (67.8, -82.9)
- added C20: 0.1uF, mouse_reach_controller:SM0402, F.Cu at (69.8, -82.9)
- added R11: 2.21k, mouse_reach_controller:SM0402, F.Cu at (71.7, -82.9)
- added R12: 2.21k, mouse_reach_controller:SM0402, F.Cu at (73.7, -82.9)
- C11: value 2.2uF -> 10uF
- C16: value 0.15uF -> 0.1uF
- C17: value 0.1uF -> 2.2uF
- C18: value 0.1uF -> 0.15uF
- C9: value 100uF_POL -> 100uF
- R7: value 2.21k -> 150k
- R8: value 2.21k -> 205k
- U8: value BSP762TXUMA1 -> DRV103; footprint mouse_reach_controller:SOIC-8_3.9x4.9mm_P1.27mm -> mouse_reach_controller:SOIC_8
- moved P4 242.3 mm to (148.6, 91.4)
- moved P3 231.9 mm to (110.5, 91.4)
- moved R1 227.7 mm to (105.4, 97.8)
- moved R2 227.7 mm to (105.4, 104.1)
- moved U2 227.7 mm to (110.5, 101.6)
- moved C3 221.9 mm to (116.8, 101.6), turned to 180 degrees
- moved C11 219.3 mm to (152.4, 78.7), turned to 0 degrees
- moved P7 204.8 mm to (213.4, 57.1)
- moved P5 203.6 mm to (186.7, 91.4)
- moved C16 203.3 mm to (165.1, 80.0), turned to 0 degrees
- moved J1 198.3 mm to (166.4, 53.3)
- moved C12 197.6 mm to (174.0, 69.8), turned to 270 degrees
- moved U9 196.5 mm to (161.3, 80.0), turned to 180 degrees
- moved L1 196.3 mm to (174.0, 73.7)
- moved U10 194.1 mm to (166.4, 73.7)
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Connections:
- C10 pad 1: /VDD -> /power_switch_driver/VBB
- C12 pad 1: Net-(C11-Pad1) -> /VDD
- C13 pad 1: /VDD -> Net-(C13-Pad1)
- C14 pad 1: /VDD -> Net-(C13-Pad1)
- C15 pad 1: /audio_controller/VEE -> /VDD
- C16 pad 1: /audio_controller/VAG -> /VDD
- C17 pad 1: /VDD -> /audio_controller/VEE
- C18 pad 1: /VDD -> /audio_controller/VAG
- D1 pad 1: /power_switch_driver/VM -> /power_switch_driver/VBB
- D1 pad 2: /GND -> /power_switch_driver/OUT
- L1 pad 2: Net-(C11-Pad1) -> Net-(C13-Pad1)
- R10 pad 2: /ENCODER_B -> /SCL
- R7 pad 1: /VDD -> Net-(R7-Pad1)
- R7 pad 2: /SDA -> /GND
- R8 pad 1: /VDD -> Net-(R8-Pad1)
- R8 pad 2: /SCL -> /GND
- R9 pad 2: /ENCODER_A -> /SDA
- T1 pad 1: /GND -> /power_switch_driver/VBB
- T1 pad 2: /power_switch_driver/VM -> /power_switch_driver/OUT
- U10 pad 5: Net-(C11-Pad1) -> Net-(C13-Pad1)
- U8 pad 1: /GND -> Net-(R7-Pad1)
- U8 pad 2: /POWER_SWITCH_ENABLE -> Net-(C11-Pad1)
- U8 pad 3: /power_switch_driver/VM -> Net-(R8-Pad1)
- U8 pad 4: (no net) -> /GND
- U8 pad 5: /power_switch_driver/VBB -> /power_switch_driver/OUT
- U8 pad 7: /power_switch_driver/VBB -> (no net)
- U8 pad 8: /power_switch_driver/VBB -> /POWER_SWITCH_ENABLE

Commit message: Added components
Parts:
- added C21: 0.1uF, mouse_reach_controller:SM0402, F.Cu at (180.8, 12.4)
- added C22: 0.1uF, mouse_reach_controller:SM0402, F.Cu at (182.8, 12.4)
- added C23: 0.1uF, mouse_reach_controller:SM0402, F.Cu at (184.8, 12.4)
- added I1: 600, mouse_reach_controller:SM1210, F.Cu at (100.3, -7.62)
- added L2: LED, mouse_reach_controller:LED_0402, F.Cu at (106.7, 74.9)
- added L3: LED, mouse_reach_controller:LED_0402, F.Cu at (86.2, 19.9)
- added L4: LED, mouse_reach_controller:LED_0402, F.Cu at (87.8, 19.9)
- added L5: LED, mouse_reach_controller:LED_0402, F.Cu at (71.4, 28.7)
- added R13: 205k, mouse_reach_controller:SM0402, F.Cu at (73.1, 28.8)
- added R14: 2.21k, mouse_reach_controller:SM0402, F.Cu at (75.6, 20.0)
- added R15: 2.21k, mouse_reach_controller:SM0402, F.Cu at (75.6, 22.9)
- added R16: 10.0k, mouse_reach_controller:SM0402, F.Cu at (85.0, 26.4)
- added R17: 10.0k, mouse_reach_controller:SM0402, F.Cu at (87.0, 26.4)
- added U13: 74LVC1G125GS, mouse_reach_controller:SOT1202, F.Cu at (180.9, 14.9)
- added U14: 74LVC1G125GS, mouse_reach_controller:SOT1202, F.Cu at (183.1, 14.9)
- added U15: 74LVC1G125GS, mouse_reach_controller:SOT1202, F.Cu at (186.8, 12.0)
- C19: value 0.1uF -> 100uF_POL; footprint mouse_reach_controller:SM0402 -> mouse_reach_controller:CP_Elec_6.3x7.7_WURTH
- CLK1: footprint mouse_reach_controller:CTS_SMD_4_7X5MM -> mouse_reach_controller:XTAL_WURTH
- L1: value 600@100MHz_1210 -> LED; footprint mouse_reach_controller:SM1210 -> mouse_reach_controller:LED_0402
- R1, R2, R3, R4: value 100 -> 750
- R10, R9: value 2.21k -> 100
- R12: value 2.21k -> 150k
- R7: value 150k -> 100
- R8: value 205k -> 100
- U11: value 74LVC1G125GS -> TMC424; footprint mouse_reach_controller:SOT1202 -> mouse_reach_controller:TQFP-100_14x14mm_P0.5mm
- moved C20 198.2 mm to (201.9, 64.8), turned to 180 degrees
- moved C19 196.1 mm to (196.8, 64.8), turned to 180 degrees
- moved R12 195.8 mm to (199.4, 67.3)
- moved R11 190.3 mm to (191.8, 64.8), turned to 180 degrees
- moved U12 159.3 mm to (199.4, 64.8), turned to 180 degrees
- moved U11 147.8 mm to (215.9, 81.3), turned to 180 degrees
- moved C10 103.7 mm to (163.8, 72.4), turned to 0 degrees
- moved L1 72.4 mm to (101.6, 74.9), turned to 180 degrees
- moved U1 48.3 mm to (88.9, 100.3)
- moved C2 48.3 mm to (90.2, 105.4)
- moved C1 41.9 mm to (86.4, 94.0)
- moved CLK1 41.9 mm to (88.9, 94.0)
- moved R2 31.8 mm to (106.7, 72.4)
- moved R1 25.7 mm to (101.6, 72.4), turned to 0 degrees
- moved C12 7.62 mm to (181.6, 69.8)
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Connections:
- C19 pad 1: /VDD -> /VCC
- D1 pad 2: /power_switch_driver/OUT -> /power_switch_driver/VAA
- D2 pad 2: /power_switch_driver/VAA -> /power_switch_driver/OUT
- L1 pad 1: /VDD -> /GND
- L1 pad 2: Net-(C13-Pad1) -> Net-(L1-Pad2)
- P7 pad 1: /encoder_interface/CHANNEL_A_BUFFERED -> /encoder_interface/CHANNEL_A_OUT
- P7 pad 3: /encoder_interface/CHANNEL_B_BUFFERED -> /encoder_interface/CHANNEL_B_OUT
- R1 pad 1: /stepper_controller/stepper_driver_interface_0/REF_A -> /BNC_A
- R1 pad 2: /stepper_controller/stepper_driver_interface_0/REF_B -> Net-(L1-Pad2)
- R10 pad 1: /VDD -> /stepper_controller/stepper_driver_interface_2/REFR_A
- R10 pad 2: /SCL -> /stepper_controller/stepper_driver_interface_2/REFR_B
- R11 pad 1: /VDD -> /power_switch_driver/VBB
- R11 pad 2: /ENCODER_A -> Net-(L5-Pad2)
- R12 pad 1: /VDD -> Net-(R12-Pad1)
- R12 pad 2: /ENCODER_B -> /GND
- R2 pad 1: /stepper_controller/stepper_driver_interface_0/REFR_A -> /BNC_B
- R2 pad 2: /stepper_controller/stepper_driver_interface_0/REFR_B -> Net-(L2-Pad2)
- R3 pad 1: /stepper_controller/stepper_driver_interface_1/REF_A -> /BNC_C
- R3 pad 2: /stepper_controller/stepper_driver_interface_1/REF_B -> Net-(L3-Pad2)
- R4 pad 1: /stepper_controller/stepper_driver_interface_1/REFR_A -> /BNC_D
- R4 pad 2: /stepper_controller/stepper_driver_interface_1/REFR_B -> Net-(L4-Pad2)
- R5 pad 1: /stepper_controller/stepper_driver_interface_2/REF_A -> /stepper_controller/stepper_driver_interface_0/REF_A
- R5 pad 2: /stepper_controller/stepper_driver_interface_2/REF_B -> /stepper_controller/stepper_driver_interface_0/REF_B
- R6 pad 1: /stepper_controller/stepper_driver_interface_2/REFR_A -> /stepper_controller/stepper_driver_interface_0/REFR_A
- R6 pad 2: /stepper_controller/stepper_driver_interface_2/REFR_B -> /stepper_controller/stepper_driver_interface_0/REFR_B
- R7 pad 1: Net-(R7-Pad1) -> /stepper_controller/stepper_driver_interface_1/REF_A
- R7 pad 2: /GND -> /stepper_controller/stepper_driver_interface_1/REF_B
- R8 pad 1: Net-(R8-Pad1) -> /stepper_controller/stepper_driver_interface_1/REFR_A
- R8 pad 2: /GND -> /stepper_controller/stepper_driver_interface_1/REFR_B
- R9 pad 1: /VDD -> /stepper_controller/stepper_driver_interface_2/REF_A
- R9 pad 2: /SDA -> /stepper_controller/stepper_driver_interface_2/REF_B
- U11 pad 1: /GND -> (no net)
- U11 pad 2: /ENCODER_A -> (no net)
- U11 pad 3: /GND -> (no net)
- U11 pad 4: /encoder_interface/CHANNEL_A_BUFFERED -> (no net)
- U11 pad 6: /VDD -> (no net)
- U12 pad 2: /ENCODER_B -> /ENCODER_A
- U12 pad 4: /encoder_interface/CHANNEL_B_BUFFERED -> (no net)
- U8 pad 1: Net-(R7-Pad1) -> Net-(R12-Pad1)
- U8 pad 3: Net-(R8-Pad1) -> Net-(R13-Pad1)
Other:
- board text added: "BNC_A"
- board text added: "BNC_B"
